Commit message: improved the code of traj_phri_deformation package, and test it in the hardware of UR

File: src/universal_robot/ur_gazebo/urdf/ur.xacro (robot description, xacro)
@@ -65,5 +65,5 @@
     <parent link="world"/>
     <child link="base_link"/>
-    <origin xyz="0 0 0" rpy="0 0 0"/>
+    <origin xyz="0 0 1" rpy="-2.526189559 0.52359878 -0.6154030943"/> <!-- E402摆放姿态 -->
   </joint>
   <link name="tool0_controller"/>
